Commit message: add camera_box to xt_dog.urdf

File: legged_gym/resources/robots/xt_dog/urdf/xt_dog.urdf (robot description, URDF)
Before this commit: robot xt_dog, 17 links, 16 joints
Links:
- added link camera_box; visual box size=0.025 0.09 0.025
Joints:
- added joint fixed_camera_box: type fixed, parent base, child camera_box, origin xyz=0 0 0 rpy=0 0 0

Commit message: modified effort from 40 to 80

File: legged_gym/resources/robots/xt_dog/urdf/xt_dog.urdf (robot description, URDF)
Before this commit: robot xt_dog, 18 links, 17 joints
Joints:
- joint FL_calf_joint: limit lower=-1.8326 upper=0.5236 effort=40 velocity=20 -> lower=-1.8326 upper=0.5236 effort=80 velocity=20
- joint FL_hip_joint: limit lower=-0.7854  upper=0.7854 effort=40 velocity=20 -> lower=-0.7854  upper=0.7854 effort=80 velocity=20
- joint FL_thigh_joint: limit lower=-1.8326 upper=1.8326 effort=40 velocity=20 -> lower=-1.8326 upper=1.8326 effort=80 velocity=20
- joint FR_calf_joint: limit lower=-1.8326 upper=0.5236 effort=40 velocity=20 -> lower=-1.8326 upper=0.5236 effort=80 velocity=20
- joint FR_hip_joint: limit lower=-0.7854  upper=0.7854 effort=40 velocity=20 -> lower=-0.7854  upper=0.7854 effort=80 velocity=20
- joint FR_thigh_joint: limit lower=-1.8326 upper=1.8326 effort=40 velocity=20 -> lower=-1.8326 upper=1.8326 effort=80 velocity=20
- joint RL_calf_joint: limit lower=-1.8326 upper=0.5236 effort=40 velocity=20 -> lower=-1.8326 upper=0.5236 effort=80 velocity=20
- joint RL_hip_joint: limit lower=-0.7854  upper=0.7854 effort=40 velocity=20 -> lower=-0.7854  upper=0.7854 effort=80 velocity=20
- joint RL_thigh_joint: limit lower=-1.8326 upper=1.8326 effort=40 velocity=20 -> lower=-1.8326 upper=1.8326 effort=80 velocity=20
- joint RR_calf_joint: limit lower=-1.8326 upper=0.5236 effort=40 velocity=20 -> lower=-1.8326 upper=0.5236 effort=80 velocity=20
- joint RR_hip_joint: limit lower=-0.7854  upper=0.7854 effort=40 velocity=20 -> lower=-0.7854  upper=0.7854 effort=80 velocity=20
- joint RR_thigh_joint: limit lower=-1.8326 upper=1.8326 effort=40 velocity=20 -> lower=-1.8326 upper=1.8326 effort=80 velocity=20
